File: Eagle/PIC32.sch (EAGLE design)
At the start: 22 parts

Commit message: Uploading revised schematic and board without ground
Parts:
- C1, C2, C3, C4: value (none) -> .1uF
- C7, C8: value (none) -> 10uF
- renumbered U$1 to REG, U$11 to .., U$2 to LEFT, U$3 to ..., U$4 to DIP_28, U$6 to ., U$7 to RESET, U$8 to USER, U$9 to RIGHT
Connections:
- net N$13 renamed A4
- net N$24 renamed B4
- removed net N$11: C3.2, DIP_28.13.VDD
- removed net N$18: ...3.GND
- new net D+: ..3.D+, DIP_28.21.D+
- new net D-: ..2.D-, DIP_28.22.D-
- new net ID: ..4.ID, DIP_28.14.USBID
- net GND: now also ...3.GND
- net V3.3: now also C3.2, DIP_28.13.VDD, DIP_28.19.VSS1, DIP_28.23.VUSB
- net VBUS: no longer DIP_28.14.USBID

Commit message: saving changes
Connections:
- net N$1 renamed B15
- net N$10 renamed A3
- net N$12 renamed A1
- net N$15 renamed VCAP
- net N$16 renamed B3
- net N$17 renamed B2
- net N$19 renamed B13
- net N$2 renamed B14
- net N$20 renamed B9
- net N$21 renamed B8
- net N$22 renamed B7
- net N$6 renamed A0
- net N$7 renamed B0
- net N$8 renamed B1
- net N$9 renamed A2
Changed lines of the file:
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@@
 </segment>
 </net>
-<net name="N$7" class="0">
+<net name="B0" class="0">
 <segment>
 <pinref part=".." gate="G$1" pin="4.B0"/>
@@
 </segment>
 </net>
-<net name="N$8" class="0">
+<net name="B1" class="0">
 <segment>
 <pinref part=".." gate="G$1" pin="5.B1"/>
@@
 </segment>
 </net>
-<net name="N$9" class="0">
+<net name="A2" class="0">
 <segment>
 <pinref part="..." gate="G$1" pin="1.OSC1"/>
@@
 </segment>
 </net>
-<net name="N$10" class="0">
+<net name="A3" class="0">
 <segment>
 <pinref part="..." gate="G$1" pin="3.OSC2"/>
@@
 </segment>
 </net>
-<net name="N$15" class="0">
+<net name="VCAP" class="0">
 <segment>
 <pinref part="DIP_28" gate="G$1" pin="20.VCAP"/>
@@
 </segment>
 </net>
-<net name="N$17" class="0">
+<net name="B2" class="0">
 <segment>
 <wire x1="40.64" y1="78.74" x2="40.64" y2="55.88" width="0.1524" layer="91"/>
@@
 </segment>
 </net>
-<net name="N$1" class="0">
+<net name="B15" class="0">
 <segment>
 <pinref part="DIP_28" gate="G$1" pin="26.B15"/>
@@
 </segment>
 </net>
-<net name="N$2" class="0">
+<net name="B14" class="0">
 <segment>
 <pinref part="RIGHT" gate="G$1" pin="2.B14"/>
@@
 </segment>
 </net>
-<net name="N$19" class="0">
+<net name="B13" class="0">
 <segment>
 <pinref part="RIGHT" gate="G$1" pin="3.B13"/>
@@
 </segment>
 </net>
-<net name="N$20" class="0">
+<net name="B9" class="0">
 <segment>
 <pinref part="RIGHT" gate="G$1" pin="4.B9"/>
@@
 </segment>
 </net>
-<net name="N$21" class="0">
+<net name="B8" class="0">
 <segment>
 <pinref part="RIGHT" gate="G$1" pin="5.B8"/>
@@
 </segment>
 </net>
-<net name="N$22" class="0">
+<net name="B7" class="0">
 <segment>
 <pinref part="RIGHT" gate="G$1" pin="6.B7"/>
@@
 </segment>
 </net>
-<net name="N$6" class="0">
+<net name="A0" class="0">
 <segment>
 <pinref part="LEFT" gate="G$1" pin="1.A0"/>
@@
 </segment>
 </net>
-<net name="N$12" class="0">
+<net name="A1" class="0">
 <segment>
 <pinref part="LEFT" gate="G$1" pin="2.A1"/>
@@
 </segment>
 </net>
-<net name="N$16" class="0">
+<net name="B3" class="0">
 <segment>
 <pinref part="LEFT" gate="G$1" pin="4.B3"/>

Commit message: updated pushbuttons and usb connection
Other:
- moved on the sheet: ...

Commit message: uploading changes to eagle files and uploading HW3 with the Gerber files
Parts:
- renumbered . to USB
Changed lines of the file:
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@@
 <part name="DIP_28" library="meche-433" deviceset="PIC32MX250F128_DIP" device=""/>
 <part name="U$5" library="meche-433" deviceset="SLIDE_SWITCH" device=""/>
-<part name="." library="meche-433" deviceset="USB_MINI_B" device=""/>
+<part name="USB" library="meche-433" deviceset="USB_MINI_B" device=""/>
 <part name="RESET" library="meche-433" deviceset="PUSH_BUTTON" device=""/>
 <part name="USER" library="meche-433" deviceset="PUSH_BUTTON" device=""/>
@@
 <instance part="DIP_28" gate="G$1" x="91.44" y="53.34"/>
 <instance part="U$5" gate="G$1" x="5.08" y="127"/>
-<instance part="." gate="G$1" x="-104.14" y="119.38" rot="MR0"/>
+<instance part="USB" gate="G$1" x="-104.14" y="119.38" rot="MR0"/>
 <instance part="RESET" gate="G$1" x="5.08" y="101.6"/>
 <instance part="USER" gate="G$1" x="10.16" y="-10.16"/>
@@
 <net name="GND" class="0">
 <segment>
-<pinref part="." gate="G$1" pin="5.GND"/>
+<pinref part="USB" gate="G$1" pin="5.GND"/>
 <wire x1="-99.06" y1="114.3" x2="-81.28" y2="114.3" width="0.1524" layer="91"/>
 <pinref part="REG" gate="G$1" pin="1.GND"/>
@@
 </segment>
 <segment>
-<pinref part="." gate="G$1" pin="1.VBUS"/>
+<pinref part="USB" gate="G$1" pin="1.VBUS"/>
 <pinref part="C1" gate="G$1" pin="1"/>
 <wire x1="-99.06" y1="124.46" x2="-81.28" y2="124.46" width="0.1524" layer="91"/>
@@
 <net name="D-" class="0">
 <segment>
-<pinref part="." gate="G$1" pin="2.D-"/>
+<pinref part="USB" gate="G$1" pin="2.D-"/>
 <wire x1="-99.06" y1="121.92" x2="-96.52" y2="121.92" width="0.1524" layer="91"/>
 </segment>
@@
 <net name="D+" class="0">
 <segment>
-<pinref part="." gate="G$1" pin="3.D+"/>
+<pinref part="USB" gate="G$1" pin="3.D+"/>
 <wire x1="-99.06" y1="119.38" x2="-96.52" y2="119.38" width="0.1524" layer="91"/>
 </segment>
@@
 <net name="ID" class="0">
 <segment>
-<pinref part="." gate="G$1" pin="4.ID"/>
+<pinref part="USB" gate="G$1" pin="4.ID"/>
 <wire x1="-99.06" y1="116.84" x2="-96.52" y2="116.84" width="0.1524" layer="91"/>
 </segment>
@@
 </sheet>
 </sheets>
+<errors>
+</errors>
 </schematic>
 </drawing>
